Commit message: brazo con gripper

File: src/CR_ROS/dobot_description/urdf/cr5_robot_with_gripper.urdf (robot description, URDF)
Before this commit: robot cr5_robot, 17 links, 16 joints
Joints:
- removed joint gripper
- added joint gripper_joint: type fixed, parent Link6, child robotiq_85_base_link, origin xyz=0 0 0 rpy=0 0 0, axis 0 0 1

Commit message: cambios en world

File: src/CR_ROS/dobot_description/urdf/cr5_robot_with_gripper.urdf (robot description, URDF)
Before this commit: robot cr5_robot, 17 links, 16 joints
Joints:
- joint joint1: limit lower=-3.14 upper=3.14 effort=0 velocity=0 -> lower=-3.14 upper=3.14 effort=300 velocity=100
- joint joint2: limit lower=-3.14 upper=3.14 effort=0 velocity=0 -> lower=-3.14 upper=3.14 effort=300 velocity=100
- joint joint3: limit lower=-2.86 upper=2.86 effort=0 velocity=0 -> lower=-2.86 upper=2.86 effort=300 velocity=100
- joint joint4: limit lower=-3.14 upper=3.14 effort=0 velocity=0 -> lower=-3.14 upper=3.14 effort=300 velocity=100
- joint joint5: limit lower=-3.14 upper=3.14 effort=0 velocity=0 -> lower=-3.14 upper=3.14 effort=300 velocity=100
- joint joint6: limit lower=-6.28 upper=6.28 effort=0 velocity=0 -> lower=-6.28 upper=6.28 effort=300 velocity=100
