Commit message: Fix de gazebo con rviz

File: src/CR_ROS/dobot_gazebo/urdf/cr5_robot_gripper.xacro (robot description, xacro)
@@ -79,4 +79,5 @@
     <axis xyz="0 0 1" />
     <limit lower="-3.14" upper="3.14" effort="300" velocity="100" />
+    <dynamics damping="1.0"/>
   </joint>
   <link name="Link2">
@@ -115,4 +116,5 @@
     <axis xyz="0 0 1" />
     <limit lower="-3.14" upper="3.14" effort="300" velocity="100" />
+    <dynamics damping="1.0"/>
   </joint>
   <link name="Link3">
@@ -151,4 +153,5 @@
     <axis  xyz="0 0 1" />
     <limit lower="-2.86"  upper="2.86"  effort="300" velocity="100" />
+    <dynamics damping="1.0"/>
   </joint>
   <link name="Link4">
@@ -186,4 +189,5 @@
     <axis xyz="0 0 1" />
     <limit lower="-3.14" upper="3.14" effort="300" velocity="100" />
+    <dynamics damping="1.0"/>
   </joint>
   <link
@@ -222,4 +226,5 @@
     <axis xyz="0 0 1" />
     <limit lower="-3.14" upper="3.14" effort="300" velocity="100" />
+    <dynamics damping="1.0"/>
   </joint>
   <link name="Link6">
